File: pcb/flick.sch (KiCad schematic (older format))
At the start: 41 parts, among them J1 DEBUG, Q1 Q_Photo_NPN, Q2 Q_NMOS_GSD, SW1 Rotary_Encoder_Switch, SW2 RESET, U1 ATSAMD21G18A-AFT, U2 AP2112M-3.3, X1 USB_C_2.0, X2 SH1106G, Y1 32.768KHz

Commit message: initial 100x60 version where I think everything works
Other:
- note added: "Mounting Holes"
- moved on the sheet: H1, H2, H3, H4
Changed lines of the file:
@@
 L Mechanical:MountingHole_Pad H1
 U 1 1 619B2F97
-P 10425 4050
-F 0 "H1" V 10425 4250 50  0000 C CNN
-F 1 "MountingHole_Pad" V 10571 4053 50  0001 C CNN
-F 2 "MountingHole:MountingHole_5mm_Pad" H 10425 4050 50  0001 C CNN
-F 3 "~" H 10425 4050 50  0001 C CNN
-	1    10425 4050
+P 10325 3700
+F 0 "H1" V 10325 3900 50  0000 C CNN
+F 1 "MountingHole_Pad" V 10471 3703 50  0001 C CNN
+F 2 "MountingHole:MountingHole_5mm_Pad" H 10325 3700 50  0001 C CNN
+F 3 "~" H 10325 3700 50  0001 C CNN
+	1    10325 3700
 	0    -1   -1   0
 $EndComp
@@
 L Mechanical:MountingHole_Pad H2
 U 1 1 619BA677
-P 10425 4225
-F 0 "H2" V 10425 4425 50  0000 C CNN
-F 1 "MountingHole_Pad" V 10571 4228 50  0001 C CNN
-F 2 "MountingHole:MountingHole_5mm_Pad" H 10425 4225 50  0001 C CNN
-F 3 "~" H 10425 4225 50  0001 C CNN
-	1    10425 4225
+P 10325 3875
+F 0 "H2" V 10325 4075 50  0000 C CNN
+F 1 "MountingHole_Pad" V 10471 3878 50  0001 C CNN
+F 2 "MountingHole:MountingHole_5mm_Pad" H 10325 3875 50  0001 C CNN
+F 3 "~" H 10325 3875 50  0001 C CNN
+	1    10325 3875
 	0    -1   -1   0
 $EndComp
@@
 L Mechanical:MountingHole_Pad H3
 U 1 1 619BAAAD
-P 10425 4400
-F 0 "H3" V 10425 4600 50  0000 C CNN
-F 1 "MountingHole_Pad" V 10571 4403 50  0001 C CNN
-F 2 "MountingHole:MountingHole_5mm_Pad" H 10425 4400 50  0001 C CNN
-F 3 "~" H 10425 4400 50  0001 C CNN
-	1    10425 4400
+P 10325 4050
+F 0 "H3" V 10325 4250 50  0000 C CNN
+F 1 "MountingHole_Pad" V 10471 4053 50  0001 C CNN
+F 2 "MountingHole:MountingHole_5mm_Pad" H 10325 4050 50  0001 C CNN
+F 3 "~" H 10325 4050 50  0001 C CNN
+	1    10325 4050
 	0    -1   -1   0
 $EndComp
@@
 L Mechanical:MountingHole_Pad H4
 U 1 1 619BAEA6
-P 10425 4575
-F 0 "H4" V 10425 4775 50  0000 C CNN
-F 1 "MountingHole_Pad" V 10571 4578 50  0001 C CNN
-F 2 "MountingHole:MountingHole_5mm_Pad" H 10425 4575 50  0001 C CNN
-F 3 "~" H 10425 4575 50  0001 C CNN
-	1    10425 4575
+P 10325 4225
+F 0 "H4" V 10325 4425 50  0000 C CNN
+F 1 "MountingHole_Pad" V 10471 4228 50  0001 C CNN
+F 2 "MountingHole:MountingHole_5mm_Pad" H 10325 4225 50  0001 C CNN
+F 3 "~" H 10325 4225 50  0001 C CNN
+	1    10325 4225
 	0    -1   -1   0
 $EndComp
@@
 L power:GND #PWR0131
 U 1 1 619BB583
-P 10575 4650
-F 0 "#PWR0131" H 10575 4400 50  0001 C CNN
-F 1 "GND" H 10580 4477 50  0000 C CNN
-F 2 "" H 10575 4650 50  0001 C CNN
-F 3 "" H 10575 4650 50  0001 C CNN
-	1    10575 4650
+P 10475 4300
+F 0 "#PWR0131" H 10475 4050 50  0001 C CNN
+F 1 "GND" H 10480 4127 50  0000 C CNN
+F 2 "" H 10475 4300 50  0001 C CNN
+F 3 "" H 10475 4300 50  0001 C CNN
+	1    10475 4300
 	1    0    0    -1
 $EndComp
 Wire Wire Line
-	10525 4575 10575 4575
+	10425 4225 10475 4225
 Wire Wire Line
-	10575 4575 10575 4650
+	10475 4225 10475 4300
 Wire Wire Line
-	10525 4400 10575 4400
+	10425 4050 10475 4050
 Wire Wire Line
-	10575 4400 10575 4575
-Connection ~ 10575 4575
+	10475 4050 10475 4225
+Connection ~ 10475 4225
 Wire Wire Line
-	10525 4225 10575 4225
+	10425 3875 10475 3875
 Wire Wire Line
-	10575 4225 10575 4400
-Connection ~ 10575 4400
+	10475 3875 10475 4050
+Connection ~ 10475 4050
 Wire Wire Line
-	10525 4050 10575 4050
+	10425 3700 10475 3700
 Wire Wire Line
-	10575 4050 10575 4225
-Connection ~ 10575 4225
+	10475 3700 10475 3875
+Connection ~ 10475 3875
 NoConn ~ 1550 5850
 NoConn ~ 1550 5950
@@
 Text Label 2750 3500 0    50   ~ 0
 VDDCORE
+Text Notes 9750 3200 0    79   ~ 0
+Mounting Holes
 $EndSCHEMATC

Commit message: Shrink to 95x50mm part 1
Mostly done with the routing, but there's still some power traces to
figure out, as well as deciding what to do with various local ground
planes (moar via stitching probably).

  * Mostly the same layout but smaller overall (to save cost at OSHPark
    which charges per square inch).
  * Remove LED driver Q2 because 7mA is actually plenty to drive an LED
    directly from the SAMD21.
  * Replace AP2112M with AP7365 voltage regulator in an SOT-25 package
    rather than chonky SOIC-8
  * Use surface mount headers for SWD debug rather than through-hole;
    makes routing slightly easier.
Parts:
- removed Q2: Q_NMOS_GSD, Package_TO_SOT_SMD:SOT-23, symbol Device:Q_NMOS_GSD
- removed U2: AP2112M-3.3, Package_SO:SO-8_3.9x4.9mm_P1.27mm, symbol Alkenta:AP2112M-3.3
- added U2: AP7365-33W, Package_TO_SOT_SMD:SOT-23-5_HandSoldering, symbol Wild:AP7365-33W
- VR1, VR2: footprint Alkenta:Potentiometer_Bourns_PTV09A-1_Single_Vertical -> Wild:Potentiometer_Bourns_PTV09A-1_Single_Vertical
- X1: footprint Alkenta:USB_C_Receptacle_GCT_USB4105 -> Wild:USB_C_Receptacle_GCT_USB4105
- X2: footprint Alkenta:GCT_FFC2B28-16_1x16-1MP_P0.5mm_Horizontal -> Wild:GCT_FFC2B28-16_1x16-1MP_P0.5mm_Horizontal; symbol Alkenta:SH1106G -> Wild:SH1106G
Connections:
- net +3V3: now also U2.5 (VOUT); no longer R3.1
- net +5V: now also U2.1 (VIN), U2.3 (EN)
- net GND: now also D1.1 (K), U2.2 (GND)
- net LED_TRIG: now also R3.1
Other:
- note added: "Green\nWP710A10LZGCK\n2mA @ 2.65 Vf"
- moved on the sheet: C10, C9, Y1
Changed lines of the file:
@@
 F 0 "X1" H 875 2425 50  0000 C CNN
 F 1 "USB_C_2.0" H 1075 2225 50  0000 C CNN
-F 2 "Alkenta:USB_C_Receptacle_GCT_USB4105" H 1375 1625 50  0001 C CNN
+F 2 "Wild:USB_C_Receptacle_GCT_USB4105" H 1375 1625 50  0001 C CNN
 F 3 "https://www.usb.org/sites/default/files/documents/usb_type-c.zip" H 1375 1625 50  0001 C CNN
 	1    1225 1625
@@
 	1    0    0    -1
 $EndComp
-$Comp
-L Alkenta:AP2112M-3.3 U2
-U 1 1 61838D89
-P 3925 1125
-F 0 "U2" H 3925 1467 50  0000 C CNN
-F 1 "AP2112M-3.3" H 3925 1376 50  0000 C CNN
-F 2 "Package_SO:SO-8_3.9x4.9mm_P1.27mm" H 3925 1450 50  0001 C CNN
-F 3 "https://www.diodes.com/assets/Datasheets/AP2112.pdf" H 3925 1225 50  0001 C CNN
-	1    3925 1125
-	1    0    0    -1
-$EndComp
 Text Notes 5950 1400 0    50   ~ 0
 VDDIN
@@
 	2575 1025 3425 1025
 $Comp
-L Device:Crystal_Small Y1
-U 1 1 6199EAC6
-P 1150 3900
-F 0 "Y1" V 1000 3900 50  0000 C CNN
-F 1 "32.768KHz" V 1300 3900 50  0000 C CNN
-F 2 "Crystal:Crystal_SMD_MicroCrystal_CC8V-T1A-2Pin_2.0x1.2mm_HandSoldering" H 1150 3900 50  0001 C CNN
-F 3 "~" H 1150 3900 50  0001 C CNN
-	1    1150 3900
-	0    1    1    0
-$EndComp
-$Comp
 L power:+3.3V #PWR0111
 U 1 1 619D1514
@@
 Text GLabel 8350 1575 2    50   Input ~ 0
 NRESET
-Wire Wire Line
-	1550 3850 1500 3850
-Wire Wire Line
-	1500 3850 1500 3800
-Wire Wire Line
-	1500 3800 1150 3800
-Wire Wire Line
-	1550 3950 1500 3950
-Wire Wire Line
-	1500 3950 1500 4000
-Wire Wire Line
-	1500 4000 1150 4000
-Wire Wire Line
-	950  3800 1150 3800
-Connection ~ 1150 3800
-Wire Wire Line
-	950  4000 1150 4000
-Connection ~ 1150 4000
-$Comp
-L power:GND #PWR0118
-U 1 1 61913AAC
-P 650 4100
-F 0 "#PWR0118" H 650 3850 50  0001 C CNN
-F 1 "GND" H 655 3927 50  0000 C CNN
-F 2 "" H 650 4100 50  0001 C CNN
-F 3 "" H 650 4100 50  0001 C CNN
-	1    650  4100
-	1    0    0    -1
-$EndComp
-Wire Wire Line
-	650  4100 650  4000
-Wire Wire Line
-	650  3800 750  3800
-Wire Wire Line
-	750  4000 650  4000
-Connection ~ 650  4000
-Wire Wire Line
-	650  4000 650  3800
-$Comp
-L Device:C_Small C10
-U 1 1 619BA2DB
-P 850 4000
-F 0 "C10" V 800 3800 50  0000 L CNN
-F 1 "15pF" V 950 3900 50  0000 L CNN
-F 2 "Capacitor_SMD:C_0603_1608Metric_Pad1.08x0.95mm_HandSolder" H 850 4000 50  0001 C CNN
-F 3 "~" H 850 4000 50  0001 C CNN
-	1    850  4000
-	0    1    1    0
-$EndComp
-$Comp
-L Device:C_Small C9
-U 1 1 619B4189
-P 850 3800
-F 0 "C9" V 900 3650 50  0000 L CNN
-F 1 "15pF" V 750 3700 50  0000 L CNN
-F 2 "Capacitor_SMD:C_0603_1608Metric_Pad1.08x0.95mm_HandSolder" H 850 3800 50  0001 C CNN
-F 3 "~" H 850 3800 50  0001 C CNN
-	1    850  3800
-	0    1    1    0
-$EndComp
 Text GLabel 1550 6250 0    50   Input ~ 0
 USB_D-
@@
 F 0 "VR2" H 5775 4029 50  0000 R CNN
 F 1 "10K" H 5775 4120 50  0000 R CNN
-F 2 "Alkenta:Potentiometer_Bourns_PTV09A-1_Single_Vertical" H 5845 4075 50  0001 C CNN
+F 2 "Wild:Potentiometer_Bourns_PTV09A-1_Single_Vertical" H 5845 4075 50  0001 C CNN
 F 3 "~" H 5845 4075 50  0001 C CNN
 	1    5845 4075
@@
 F 0 "VR1" H 4575 4429 50  0000 R CNN
 F 1 "10K" H 4575 4520 50  0000 R CNN
-F 2 "Alkenta:Potentiometer_Bourns_PTV09A-1_Single_Vertical" H 4645 4475 50  0001 C CNN
+F 2 "Wild:Potentiometer_Bourns_PTV09A-1_Single_Vertical" H 4645 4475 50  0001 C CNN
 F 3 "~" H 4645 4475 50  0001 C CNN
 	1    4645 4475
@@
 	0    -1   -1   0
 $EndComp
-$Comp
-L Alkenta:SH1106G X2
-U 1 1 61855B25
-P 8250 4325
-F 0 "X2" H 8250 5000 50  0000 C CNN
-F 1 "SH1106G" H 8250 4909 50  0000 C CNN
-F 2 "Alkenta:GCT_FFC2B28-16_1x16-1MP_P0.5mm_Horizontal" H 7950 4575 50  0001 C CNN
-F 3 "" H 7950 4575 50  0001 C CNN
-	1    8250 4325
-	1    0    0    -1
-$EndComp
 Text GLabel 7800 4125 0    50   Input ~ 0
 OLED_CS
@@
 	1    0    0    -1
 $EndComp
-Text GLabel 4650 6450 0    50   Input ~ 0
+Text GLabel 4900 5700 0    50   Input ~ 0
 LED_TRIG
 Text GLabel 1550 5450 0    50   Input ~ 0
@@
 Text GLabel 1550 4750 0    50   Input ~ 0
 OLED_RESET
-$Comp
-L power:+3.3V #PWR0127
-U 1 1 619CC6B0
-P 4950 5750
-F 0 "#PWR0127" H 4950 5600 50  0001 C CNN
-F 1 "+3.3V" H 4965 5923 50  0000 C CNN
-F 2 "" H 4950 5750 50  0001 C CNN
-F 3 "" H 4950 5750 50  0001 C CNN
-	1    4950 5750
-	1    0    0    -1
-$EndComp
 $Comp
 L Device:Rotary_Encoder_Switch SW1
@@
 NoConn ~ 1550 5150
 $Comp
-L Device:Q_NMOS_GSD Q2
-U 1 1 61A68A78
-P 4850 6450
-F 0 "Q2" H 5054 6496 50  0000 L CNN
-F 1 "Q_NMOS_GSD" H 5054 6405 50  0000 L CNN
-F 2 "Package_TO_SOT_SMD:SOT-23" H 5050 6550 50  0001 C CNN
-F 3 "~" H 4850 6450 50  0001 C CNN
-	1    4850 6450
-	1    0    0    -1
-$EndComp
-$Comp
 L power:GND #PWR01
 U 1 1 61A7C612
-P 4950 6650
-F 0 "#PWR01" H 4950 6400 50  0001 C CNN
-F 1 "GND" H 4955 6477 50  0000 C CNN
-F 2 "" H 4950 6650 50  0001 C CNN
-F 3 "" H 4950 6650 50  0001 C CNN
-	1    4950 6650
+P 4950 6250
+F 0 "#PWR01" H 4950 6000 50  0001 C CNN
+F 1 "GND" H 4955 6077 50  0000 C CNN
+F 2 "" H 4950 6250 50  0001 C CNN
+F 3 "" H 4950 6250 50  0001 C CNN
+	1    4950 6250
 	1    0    0    -1
 $EndComp
@@
 Text Notes 9750 3200 0    79   ~ 0
 Mounting Holes
+Wire Wire Line
+	4950 5750 4950 5700
+Wire Wire Line
+	4950 5700 4900 5700
+Text Notes 4850 6150 2    50   ~ 0
+Green\nWP710A10LZGCK\n2mA @ 2.65 Vf
+$Comp
+L Wild:AP7365-33W U2
+U 1 1 61905D50
+P 3925 1125
+F 0 "U2" H 3925 1467 50  0000 C CNN
+F 1 "AP7365-33W" H 3925 1376 50  0000 C CNN
+F 2 "Package_TO_SOT_SMD:SOT-23-5_HandSoldering" H 3925 1450 50  0001 C CNN
+F 3 "https://www.diodes.com/assets/Datasheets/products_inactive_data/AP7365.pdf" H 3925 1225 50  0001 C CNN
+	1    3925 1125
+	1    0    0    -1
+$EndComp
+$Comp
+L Wild:SH1106G X2
+U 1 1 61855B25
+P 8250 4325
+F 0 "X2" H 8250 5000 50  0000 C CNN
+F 1 "SH1106G" H 8250 4909 50  0000 C CNN
+F 2 "Wild:GCT_FFC2B28-16_1x16-1MP_P0.5mm_Horizontal" H 7950 4575 50  0001 C CNN
+F 3 "" H 7950 4575 50  0001 C CNN
+	1    8250 4325
+	1    0    0    -1
+$EndComp
+$Comp
+L Device:Crystal_Small Y1
+U 1 1 6199EAC6
+P 1275 3900
+F 0 "Y1" V 1125 3900 50  0000 C CNN
+F 1 "32.768KHz" V 1425 3900 50  0000 C CNN
+F 2 "Crystal:Crystal_SMD_MicroCrystal_CC8V-T1A-2Pin_2.0x1.2mm_HandSoldering" H 1275 3900 50  0001 C CNN
+F 3 "~" H 1275 3900 50  0001 C CNN
+	1    1275 3900
+	0    1    1    0
+$EndComp
+Wire Wire Line
+	1075 3800 1275 3800
+Wire Wire Line
+	1075 4000 1275 4000
+$Comp
+L power:GND #PWR0118
+U 1 1 61913AAC
+P 775 4100
+F 0 "#PWR0118" H 775 3850 50  0001 C CNN
+F 1 "GND" H 780 3927 50  0000 C CNN
+F 2 "" H 775 4100 50  0001 C CNN
+F 3 "" H 775 4100 50  0001 C CNN
+	1    775  4100
+	1    0    0    -1
+$EndComp
+Wire Wire Line
+	775  4100 775  4000
+Wire Wire Line
+	775  3800 875  3800
+Wire Wire Line
+	875  4000 775  4000
+Connection ~ 775  4000
+Wire Wire Line
+	775  4000 775  3800
+$Comp
+L Device:C_Small C10
+U 1 1 619BA2DB
+P 975 4000
+F 0 "C10" V 925 3800 50  0000 L CNN
+F 1 "15pF" V 1075 3900 50  0000 L CNN
+F 2 "Capacitor_SMD:C_0603_1608Metric_Pad1.08x0.95mm_HandSolder" H 975 4000 50  0001 C CNN
+F 3 "~" H 975 4000 50  0001 C CNN
+	1    975  4000
+	0    1    1    0
+$EndComp
+$Comp
+L Device:C_Small C9
+U 1 1 619B4189
+P 975 3800
+F 0 "C9" V 1025 3650 50  0000 L CNN
+F 1 "15pF" V 875 3700 50  0000 L CNN
+F 2 "Capacitor_SMD:C_0603_1608Metric_Pad1.08x0.95mm_HandSolder" H 975 3800 50  0001 C CNN
+F 3 "~" H 975 3800 50  0001 C CNN
+	1    975  3800
+	0    1    1    0
+$EndComp
+Wire Wire Line
+	1550 3850 1475 3850
+Wire Wire Line
+	1475 3850 1475 3800
+Wire Wire Line
+	1475 3800 1275 3800
+Connection ~ 1275 3800
+Wire Wire Line
+	1275 4000 1475 4000
+Wire Wire Line
+	1475 4000 1475 3950
+Wire Wire Line
+	1475 3950 1550 3950
+Connection ~ 1275 4000
 $EndSCHEMATC

Commit message: draft of v1 shrink complete
Add test points, flip the phototransistor footprint around (so
anode/cathode is consistent with standard LEDs), finish routing power
and stuff.

TODO: Add silkscreen text/graphics, verify I can actually order
everything in the BOM, double-check everything before production.
Parts:
- added TP1: GND, Wild:TestPoint_THTPad_D1.6mm_Drill1.0mm, symbol Connector:TestPoint
- added TP2: VCC, Wild:TestPoint_THTPad_D1.6mm_Drill1.0mm, symbol Connector:TestPoint
- added TP3: VCCA, Wild:TestPoint_THTPad_D1.6mm_Drill1.0mm, symbol Connector:TestPoint
- added TP4: THRSH, Wild:TestPoint_THTPad_D1.6mm_Drill1.0mm, symbol Connector:TestPoint
- added TP5: VAL, Wild:TestPoint_THTPad_D1.6mm_Drill1.0mm, symbol Connector:TestPoint
- Q1: symbol Device:Q_Photo_NPN -> Device:Q_Photo_NPN_EC
Connections:
- net +3.3VA: now also Q1.2 (C), TP3.1; no longer Q1.1 (C)
- net +3V3: now also TP2.1
- net GND: now also TP1.1
- net PHOTO_THRESH: now also TP4.1
- net PHOTO_VAL: now also Q1.1 (E), TP5.1; no longer Q1.2 (E)
Other:
- note added: "Test Points"
- moved on the sheet: H1, H2, H3, H4
Changed lines of the file:
@@
 Connection ~ 4325 1475
 $Comp
-L Device:Q_Photo_NPN Q1
+L Device:Q_Photo_NPN_EC Q1
 U 1 1 619646AD
 P 4695 3975
@@
 L Mechanical:MountingHole_Pad H1
 U 1 1 619B2F97
-P 10325 3700
-F 0 "H1" V 10325 3900 50  0000 C CNN
-F 1 "MountingHole_Pad" V 10471 3703 50  0001 C CNN
-F 2 "MountingHole:MountingHole_5mm_Pad" H 10325 3700 50  0001 C CNN
-F 3 "~" H 10325 3700 50  0001 C CNN
-	1    10325 3700
+P 10375 5650
+F 0 "H1" V 10375 5850 50  0000 C CNN
+F 1 "MountingHole_Pad" V 10521 5653 50  0001 C CNN
+F 2 "MountingHole:MountingHole_5mm_Pad" H 10375 5650 50  0001 C CNN
+F 3 "~" H 10375 5650 50  0001 C CNN
+	1    10375 5650
 	0    -1   -1   0
 $EndComp
@@
 L Mechanical:MountingHole_Pad H2
 U 1 1 619BA677
-P 10325 3875
-F 0 "H2" V 10325 4075 50  0000 C CNN
-F 1 "MountingHole_Pad" V 10471 3878 50  0001 C CNN
-F 2 "MountingHole:MountingHole_5mm_Pad" H 10325 3875 50  0001 C CNN
-F 3 "~" H 10325 3875 50  0001 C CNN
-	1    10325 3875
+P 10375 5825
+F 0 "H2" V 10375 6025 50  0000 C CNN
+F 1 "MountingHole_Pad" V 10521 5828 50  0001 C CNN
+F 2 "MountingHole:MountingHole_5mm_Pad" H 10375 5825 50  0001 C CNN
+F 3 "~" H 10375 5825 50  0001 C CNN
+	1    10375 5825
 	0    -1   -1   0
 $EndComp
@@
 L Mechanical:MountingHole_Pad H3
 U 1 1 619BAAAD
-P 10325 4050
-F 0 "H3" V 10325 4250 50  0000 C CNN
-F 1 "MountingHole_Pad" V 10471 4053 50  0001 C CNN
-F 2 "MountingHole:MountingHole_5mm_Pad" H 10325 4050 50  0001 C CNN
-F 3 "~" H 10325 4050 50  0001 C CNN
-	1    10325 4050
+P 10375 6000
+F 0 "H3" V 10375 6200 50  0000 C CNN
+F 1 "MountingHole_Pad" V 10521 6003 50  0001 C CNN
+F 2 "MountingHole:MountingHole_5mm_Pad" H 10375 6000 50  0001 C CNN
+F 3 "~" H 10375 6000 50  0001 C CNN
+	1    10375 6000
 	0    -1   -1   0
 $EndComp
@@
 L Mechanical:MountingHole_Pad H4
 U 1 1 619BAEA6
-P 10325 4225
-F 0 "H4" V 10325 4425 50  0000 C CNN
-F 1 "MountingHole_Pad" V 10471 4228 50  0001 C CNN
-F 2 "MountingHole:MountingHole_5mm_Pad" H 10325 4225 50  0001 C CNN
-F 3 "~" H 10325 4225 50  0001 C CNN
-	1    10325 4225
+P 10375 6175
+F 0 "H4" V 10375 6375 50  0000 C CNN
+F 1 "MountingHole_Pad" V 10521 6178 50  0001 C CNN
+F 2 "MountingHole:MountingHole_5mm_Pad" H 10375 6175 50  0001 C CNN
+F 3 "~" H 10375 6175 50  0001 C CNN
+	1    10375 6175
 	0    -1   -1   0
 $EndComp
@@
 L power:GND #PWR0131
 U 1 1 619BB583
-P 10475 4300
-F 0 "#PWR0131" H 10475 4050 50  0001 C CNN
-F 1 "GND" H 10480 4127 50  0000 C CNN
-F 2 "" H 10475 4300 50  0001 C CNN
-F 3 "" H 10475 4300 50  0001 C CNN
-	1    10475 4300
-	1    0    0    -1
-$EndComp
-Wire Wire Line
-	10425 4225 10475 4225
-Wire Wire Line
-	10475 4225 10475 4300
-Wire Wire Line
-	10425 4050 10475 4050
-Wire Wire Line
-	10475 4050 10475 4225
-Connection ~ 10475 4225
-Wire Wire Line
-	10425 3875 10475 3875
-Wire Wire Line
-	10475 3875 10475 4050
-Connection ~ 10475 4050
-Wire Wire Line
-	10425 3700 10475 3700
-Wire Wire Line
-	10475 3700 10475 3875
-Connection ~ 10475 3875
+P 10525 6250
+F 0 "#PWR0131" H 10525 6000 50  0001 C CNN
+F 1 "GND" H 10530 6077 50  0000 C CNN
+F 2 "" H 10525 6250 50  0001 C CNN
+F 3 "" H 10525 6250 50  0001 C CNN
+	1    10525 6250
+	1    0    0    -1
+$EndComp
+Wire Wire Line
+	10475 6175 10525 6175
+Wire Wire Line
+	10525 6175 10525 6250
+Wire Wire Line
+	10475 6000 10525 6000
+Wire Wire Line
+	10525 6000 10525 6175
+Connection ~ 10525 6175
+Wire Wire Line
+	10475 5825 10525 5825
+Wire Wire Line
+	10525 5825 10525 6000
+Connection ~ 10525 6000
+Wire Wire Line
+	10475 5650 10525 5650
+Wire Wire Line
+	10525 5650 10525 5825
+Connection ~ 10525 5825
 NoConn ~ 1550 5850
 NoConn ~ 1550 5950
@@
 VDDCORE
 Text Notes 9750 3200 0    79   ~ 0
-Mounting Holes
+Test Points
 Wire Wire Line
 	4950 5750 4950 5700
@@
 	1475 3950 1550 3950
 Connection ~ 1275 4000
+$Comp
+L Connector:TestPoint TP1
+U 1 1 618B8234
+P 10400 3450
+F 0 "TP1" V 10354 3638 50  0000 L CNN
+F 1 "GND" V 10445 3638 50  0000 L CNN
+F 2 "Wild:TestPoint_THTPad_D1.6mm_Drill1.0mm" H 10600 3450 50  0001 C CNN
+F 3 "~" H 10600 3450 50  0001 C CNN
+	1    10400 3450
+	0    1    1    0
+$EndComp
+$Comp
+L power:GND #PWR0127
+U 1 1 618BCF7E
+P 10400 3450
+F 0 "#PWR0127" H 10400 3200 50  0001 C CNN
+F 1 "GND" V 10400 3250 50  0000 C CNN
+F 2 "" H 10400 3450 50  0001 C CNN
+F 3 "" H 10400 3450 50  0001 C CNN
+	1    10400 3450
+	0    1    1    0
+$EndComp
+$Comp
+L Connector:TestPoint TP2
+U 1 1 618BD7D7
+P 10400 3700
+F 0 "TP2" V 10354 3888 50  0000 L CNN
+F 1 "VCC" V 10445 3888 50  0000 L CNN
+F 2 "Wild:TestPoint_THTPad_D1.6mm_Drill1.0mm" H 10600 3700 50  0001 C CNN
+F 3 "~" H 10600 3700 50  0001 C CNN
+	1    10400 3700
+	0    1    1    0
+$EndComp
+$Comp
+L power:+3.3V #PWR0132
+U 1 1 618C3128
+P 10400 3700
+F 0 "#PWR0132" H 10400 3550 50  0001 C CNN
+F 1 "+3.3V" V 10400 3950 50  0000 C CNN
+F 2 "" H 10400 3700 50  0001 C CNN
+F 3 "" H 10400 3700 50  0001 C CNN
+	1    10400 3700
+	0    -1   -1   0
+$EndComp
+$Comp
+L Connector:TestPoint TP3
+U 1 1 618CAF32
+P 10400 3950
+F 0 "TP3" V 10354 4138 50  0000 L CNN
+F 1 "VCCA" V 10445 4138 50  0000 L CNN
+F 2 "Wild:TestPoint_THTPad_D1.6mm_Drill1.0mm" H 10600 3950 50  0001 C CNN
+F 3 "~" H 10600 3950 50  0001 C CNN
+	1    10400 3950
+	0    1    1    0
+$EndComp
+$Comp
+L power:+3.3VA #PWR0133
+U 1 1 618CBAA3
+P 10400 3950
+F 0 "#PWR0133" H 10400 3800 50  0001 C CNN
+F 1 "+3.3VA" V 10415 4077 50  0000 L CNN
+F 2 "" H 10400 3950 50  0001 C CNN
+F 3 "" H 10400 3950 50  0001 C CNN
+	1    10400 3950
+	0    -1   -1   0
+$EndComp
+$Comp
+L Connector:TestPoint TP4
+U 1 1 618CC9D7
+P 10400 4200
+F 0 "TP4" V 10354 4388 50  0000 L CNN
+F 1 "THRSH" V 10445 4388 50  0000 L CNN
+F 2 "Wild:TestPoint_THTPad_D1.6mm_Drill1.0mm" H 10600 4200 50  0001 C CNN
+F 3 "~" H 10600 4200 50  0001 C CNN
+	1    10400 4200
+	0    1    1    0
+$EndComp
+Text GLabel 10400 4200 0    50   Input ~ 0
+PHOTO_THRESH
+$Comp
+L Connector:TestPoint TP5
+U 1 1 618D25ED
+P 10400 4450
+F 0 "TP5" V 10354 4638 50  0000 L CNN
+F 1 "VAL" V 10445 4638 50  0000 L CNN
+F 2 "Wild:TestPoint_THTPad_D1.6mm_Drill1.0mm" H 10600 4450 50  0001 C CNN
+F 3 "~" H 10600 4450 50  0001 C CNN
+	1    10400 4450
+	0    1    1    0
+$EndComp
+Text GLabel 10400 4450 0    50   Input ~ 0
+PHOTO_VAL
+Text Notes 9750 5400 0    79   ~ 0
+Mounting Holes
 $EndSCHEMATC
