File: pcb/flick.sch (KiCad schematic (older format))
At the start: 45 parts, among them J1 DEBUG, Q1 Q_Photo_NPN, SW1 Rotary_Encoder_Switch, SW2 RESET, U1 ATSAMD21G18A-AFT, U2 AP7365-33W, X1 USB_C_2.0, X2 SH1106G, Y1 32.768KHz

Commit message: Flick v1 PCB Rev A Final
Here we go, I'm gonna send this to OSH Park and hope it works. Minor
layout tweaks, add silkscreen decorations, and double-check everything.
Parts:
- added X3: SH1106G_Screen, Wild:SH1106G_SCREEN, symbol Wild:SH1106G_Screen
- C1, C14, C15, C6: DigiKey PN (none) -> 1276-1026-1-ND; DigiKey URL (none) -> https://www.digikey.com/en/products/detail/samsung-electro-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
- C10, C9: DigiKey PN (none) -> 1292-1487-1-ND; DigiKey URL (none) -> https://www.digikey.com/en/products/detail/walsin-technolog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
- C11, C3, C4, C5, C8: DigiKey PN (none) -> 1276-1935-1-ND; DigiKey URL (none) -> https://www.digikey.com/en/products/detail/samsung-electro-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
- C12, C13, C2, C7: DigiKey PN (none) -> 1276-2893-1-ND; DigiKey URL (none) -> https://www.digikey.com/en/products/detail/samsung-electro-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
- D1: DigiKey PN (none) -> 754-1915-ND; DigiKey URL (none) -> https://www.digikey.com/en/products/detail/kingbright/WP710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
- F1: DigiKey PN (none) -> 507-1800-1-ND; DigiKey URL (none) -> https://www.digikey.com/en/products/detail/bel-fuse-inc/0ZC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
- FB1: value 50ohm @ 20MHz -> 220ohm @ 100MHz; DigiKey PN (none) -> A103650CT-ND; DigiKey URL (none) -> https://www.digikey.com/en/products/detail/te-connectivity-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
- J1: DigiKey PN (none) -> S9012E-05-ND; DigiKey URL (none) -> https://www.digikey.com/en/products/detail/sullins-connecto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
- Q1: DigiKey PN (none) -> 1528-2545-ND; DigiKey URL (none) -> https://www.digikey.com/en/products/detail/adafruit-industr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
- R1, R2, R4: DigiKey PN (none) -> RMCF0603FT5K10CT-ND; DigiKey URL (none) -> https://www.digikey.com/en/products/detail/stackpole-electr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
- R3, R5: DigiKey PN (none) -> RMCF0805FT330RCT-ND; DigiKey URL (none) -> https://www.digikey.com/en/products/detail/stackpole-electr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
- R6: DigiKey PN (none) -> RMCF0805FT10K0CT-ND; DigiKey URL (none) -> https://www.digikey.com/en/products/detail/stackpole-electr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
- R7: DigiKey PN (none) -> RMCF0603FT680KCT-ND; DigiKey URL (none) -> https://www.digikey.com/en/products/detail/stackpole-electr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
- SW1: footprint Alkenta:RotaryEncoder_Bourns_PEC11L-Switch_Vertical_H20mm -> Wild:RotaryEncoder_Bourns_PEC11L-Switch_Vertical_H20mm; DigiKey PN (none) -> 118-PEC11L-4120K-S0020-ND; DigiKey URL (none) -> https://www.digikey.com/en/products/detail/bourns-inc/PEC11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
- SW2: DigiKey PN (none) -> CKN11907CT-ND; DigiKey URL (none) -> https://www.digikey.com/en/products/detail/c-k/PTS645SH43SM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
- U1: value ATSAMD21G18A-AFT -> ATSAMD21G18A-A; DigiKey PN (none) -> ATSAMD21G18A-AFTCT-ND; DigiKey URL (none) -> https://www.digikey.com/en/products/detail/microchip-techno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
- U2: DigiKey PN (none) -> AP7365-33WG-7DICT-ND; DigiKey URL (none) -> https://www.digikey.com/en/products/detail/diodes-incorpora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
- VR1, VR2: DigiKey PN (none) -> PTV09A-4020S-B103-ND; DigiKey URL (none) -> https://www.digikey.com/en/products/detail/bourns-inc/PTV09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
- X1: DigiKey PN (none) -> 2073-USB4105-GF-ACT-ND; DigiKey URL (none) -> https://www.digikey.com/en/products/detail/gct/USB4105-GF-A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
- X2: DigiKey PN (none) -> 2073-FFC2B28-16-GCT-ND; DigiKey URL (none) -> https://www.digikey.com/en/products/detail/gct/FFC2B28-16-G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
- Y1: DigiKey PN (none) -> 2195-CM8V-T1A-32.768KHZ-12.5PF-20PPM-TA-QCCT-ND; DigiKey URL (none) -> https://www.digikey.com/en/products/detail/micro-crystal-ag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
Other:
- note added: "Analog"
- note added: "Datasheet suggests 1K pullup on SWCLK,\nbut neither SparkFun nor Adafruit boards\ninclude one so it's probably safe to exclude"
- note added: "No separate GNDANA net,\njust tie directly to GND"
- note added: "Peripherals:\n\nSERCOM1 as SPI for OLED screen (with software CS)\n\nAC0 analog comparator, using two external inputs. Must use AC0\nrather than AC1 so that the LED can be the hardware output.\n\nAvoid using analog pins for digital signals: PA00-PA07, PB02-PB09,\nthey're supplied by VDDANA."
- note added: "Pin Functions"
- note added: "RC filter circuit suggested\nby SAMD21 datasheet"
- note added: "Sensitivity pot"
- note added: "Threshold pot"
- note added: "Virtual Component for screen\nfootprint and BOM only"
- moved on the sheet: C12, C13, C14, C15, D1, H1, H2, H3, H4, R3, R4, R7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
